Commit message: adding 2 more configurations for the 440LE
HCG: inverted gearboxes for high ground clearance

ECI: Extended track width and high ground clearance

File: segway_description/urdf/RMP_440LE/rmp.urdf.xacro (robot description, xacro)
@@ -27,10 +27,14 @@
     <xacro:include filename="$(find segway_description)/urdf/segway_components/single_spacer.urdf.xacro" />
     <xacro:include filename="$(find segway_description)/urdf/segway_components/std_gearbox_chassis.urdf.xacro" />
+    <xacro:include filename="$(find segway_description)/urdf/segway_components/inv_double_spacer.urdf.xacro" />
+    <xacro:include filename="$(find segway_description)/urdf/segway_components/inv_gearbox_chassis.urdf.xacro" />
+    <xacro:include filename="$(find segway_description)/urdf/segway_components/inv_gearbox_ext_spacer_chassis.urdf.xacro" />
+    <xacro:include filename="$(find segway_description)/urdf/segway_components/eci_440_spacer.urdf.xacro" />
     <xacro:include filename="$(find segway_description)/urdf/segway_components/large_enclosure.urdf.xacro" />
     <xacro:include filename="$(find segway_description)/urdf/accessories.urdf.xacro" />
     <property name="M_PI" value="3.14159"/>
     <!-- Wheel Mounting Positions -->
-    <xacro:property name="wheel_track" value="0.66067" />
-    <xacro:property name="wheel_vertical_offset" value="0.08255015" />
+    <xacro:property name="wheel_track" value="$(optenv SEGWAY_440LE_WHEEL_TRACK 0.66067)" />
+    <xacro:property name="wheel_vertical_offset" value="$(optenv SEGWAY_440LE_WHEEL_OFFSET 0.08255015)" />
     <xacro:property name="wheel_base" value="0.57150" />
     <!-- Wheel Properties -->
@@ -53,19 +57,55 @@
             <child link="base_chassis_link" />
         </joint>
-        <link name="inertial_collision_link">
-			<inertial>
-				<mass value="91.028000" />
-				<origin xyz="-0.033312 -0.001314 0.043167" rpy="${-M_PI / 2.0} 0 0"/>
-				<inertia ixx="2.625517"  ixy="0.032260"  ixz="-0.019196"
-                         iyx="0.032260"  iyy="8.046165"  iyz="-0.006618"
-                         izx="-0.019196" izy="-0.006618" izz="9.655358" />
-			</inertial>
-            <collision>
-                <origin xyz="0 0 0" rpy="${-M_PI / 2.0} 0 0" />
-				<geometry>
-					<mesh filename="package://segway_description/meshes/collision/RMP440LE_chassis_collision.stl" />
-				</geometry>
-			</collision>
-		</link>
+        <xacro:if value="$(optenv SEGWAY_440_LE_STD true)">
+            <link name="inertial_collision_link">
+			    <inertial>
+				    <mass value="91.028000" />
+				    <origin xyz="-0.033312 -0.001314 0.043167" rpy="${-M_PI / 2.0} 0 0"/>
+				    <inertia ixx="2.625517"  ixy="0.032260"  ixz="-0.019196"
+                             iyx="0.032260"  iyy="8.046165"  iyz="-0.006618"
+                             izx="-0.019196" izy="-0.006618" izz="9.655358" />
+			    </inertial>
+                <collision>
+                    <origin xyz="0 0 0" rpy="${-M_PI / 2.0} 0 0" />
+				    <geometry>
+					    <mesh filename="package://segway_description/meshes/collision/RMP440LE_chassis_collision.stl" />
+				    </geometry>
+			    </collision>
+		    </link>
+		</xacro:if>
+        <xacro:if value="$(optenv SEGWAY_440_LE_HCG false)">
+            <link name="inertial_collision_link">
+			    <inertial>
+				    <mass value="91.028000" />
+				    <origin xyz="-0.033312 -0.001314 0.043167" rpy="${-M_PI / 2.0} 0 0"/>
+				    <inertia ixx="2.625517"  ixy="0.032260"  ixz="-0.019196"
+                             iyx="0.032260"  iyy="8.046165"  iyz="-0.006618"
+                             izx="-0.019196" izy="-0.006618" izz="9.655358" />
+			    </inertial>
+                <collision>
+                    <origin xyz="0 0 0" rpy="${-M_PI / 2.0} 0 0" />
+				    <geometry>
+					    <mesh filename="package://segway_description/meshes/collision/440LE_hcg_collision.stl" />
+				    </geometry>
+			    </collision>
+		    </link>
+		</xacro:if>
+        <xacro:if value="$(optenv SEGWAY_440_LE_ECI false)">
+            <link name="inertial_collision_link">
+			    <inertial>
+				    <mass value="91.028000" />
+				    <origin xyz="-0.033312 -0.001314 0.043167" rpy="${-M_PI / 2.0} 0 0"/>
+				    <inertia ixx="2.625517"  ixy="0.032260"  ixz="-0.019196"
+                             iyx="0.032260"  iyy="8.046165"  iyz="-0.006618"
+                             izx="-0.019196" izy="-0.006618" izz="9.655358" />
+			    </inertial>
+                <collision>
+                    <origin xyz="0 0 0" rpy="0 0 0" />
+				    <geometry>
+					    <mesh filename="package://segway_description/meshes/collision/440ECI_extented_chassis_collision.stl" />
+				    </geometry>
+			    </collision>
+		    </link>
+		</xacro:if>
 		<joint name="inertial_collision_joint" type="fixed" >
 		    <parent link="base_chassis_link" />
@@ -73,10 +113,30 @@
 		</joint>
         <!--Chassis -->
-        <xacro:std_gearbox_chassis chassis_prefix="front" parent="base_chassis_link">
-            <origin xyz="${wheel_base/2} 0 0" rpy="0 0 ${M_PI}" />
-        </xacro:std_gearbox_chassis>
-        <xacro:std_gearbox_chassis chassis_prefix="rear" parent="base_chassis_link">
-            <origin xyz="${-wheel_base/2} 0 0" rpy="0 0 0" />
-        </xacro:std_gearbox_chassis>
+        <xacro:if value="$(optenv SEGWAY_440_LE_STD true)">
+            <xacro:std_gearbox_chassis chassis_prefix="front" parent="base_chassis_link">
+                <origin xyz="${wheel_base/2} 0 0" rpy="0 0 ${M_PI}" />
+            </xacro:std_gearbox_chassis>
+            <xacro:std_gearbox_chassis chassis_prefix="rear" parent="base_chassis_link">
+                <origin xyz="${-wheel_base/2} 0 0" rpy="0 0 0" />
+            </xacro:std_gearbox_chassis>
+        </xacro:if>
+        <xacro:if value="$(optenv SEGWAY_440_LE_HCG false)">
+            <!--Chassis -->
+            <xacro:inv_gearbox_chassis chassis_prefix="front" parent="base_chassis_link">
+                <origin xyz="${wheel_base/2} 0 0" rpy="0 0 ${M_PI}" />
+            </xacro:inv_gearbox_chassis>
+            <xacro:inv_gearbox_chassis chassis_prefix="rear" parent="base_chassis_link">
+                <origin xyz="${-wheel_base/2} 0 0" rpy="0 0 0" />
+            </xacro:inv_gearbox_chassis>
+        </xacro:if>
+        <xacro:if value="$(optenv SEGWAY_440_LE_ECI false)">
+            <!--Chassis -->
+            <xacro:inv_gearbox_ext_spacer_chassis chassis_prefix="front" parent="base_chassis_link">
+                <origin xyz="${wheel_base/2} 0 0" rpy="0 0 ${M_PI}" />
+            </xacro:inv_gearbox_ext_spacer_chassis>
+            <xacro:inv_gearbox_ext_spacer_chassis chassis_prefix="rear" parent="base_chassis_link">
+                <origin xyz="${-wheel_base/2} 0 0" rpy="0 0 0" />
+            </xacro:inv_gearbox_ext_spacer_chassis>
+        </xacro:if>
         <!-- Segway BSA Link (sign convention applied at embedded level)-->
         <link name="bsa_link"/>
@@ -101,16 +161,31 @@
         </xacro:battery>
         <!--Gearbox Spacers -->
-        <xacro:single_spacer spacer_prefix="front_left" parent="base_chassis_link">
-            <origin xyz="${wheel_base/2} 0.19582 0.00665" rpy="0 0 0" />
-        </xacro:single_spacer>
-        <xacro:single_spacer spacer_prefix="front_right" parent="base_chassis_link">
-            <origin xyz="${wheel_base/2} -0.19582 0.00665" rpy="0 0 ${M_PI}" />
-        </xacro:single_spacer>
-        <xacro:single_spacer spacer_prefix="rear_left" parent="base_chassis_link">
-            <origin xyz="${-wheel_base/2} 0.19582 0.00665" rpy="0 0 0" />
-        </xacro:single_spacer>
-        <xacro:single_spacer spacer_prefix="rear_right" parent="base_chassis_link">
-            <origin xyz="${-wheel_base/2} -0.19582 0.00665" rpy="0 0 ${M_PI}" />
-        </xacro:single_spacer>
+        <xacro:if value="$(optenv SEGWAY_440_LE_STD true)">
+            <xacro:single_spacer spacer_prefix="front_left" parent="base_chassis_link">
+                <origin xyz="${wheel_base/2} 0.19582 0.00665" rpy="0 0 0" />
+            </xacro:single_spacer>
+            <xacro:single_spacer spacer_prefix="front_right" parent="base_chassis_link">
+                <origin xyz="${wheel_base/2} -0.19582 0.00665" rpy="0 0 ${M_PI}" />
+            </xacro:single_spacer>
+            <xacro:single_spacer spacer_prefix="rear_left" parent="base_chassis_link">
+                <origin xyz="${-wheel_base/2} 0.19582 0.00665" rpy="0 0 0" />
+            </xacro:single_spacer>
+            <xacro:single_spacer spacer_prefix="rear_right" parent="base_chassis_link">
+                <origin xyz="${-wheel_base/2} -0.19582 0.00665" rpy="0 0 ${M_PI}" />
+            </xacro:single_spacer>
+        </xacro:if>
+        <xacro:if value="$(optenv SEGWAY_440_LE_HCG false)">
+            <xacro:inv_double_spacer spacer_prefix="left" parent="base_chassis_link">
+                <origin xyz="0 0.19582 0" rpy="0 0 0" />
+            </xacro:inv_double_spacer>
+            <xacro:inv_double_spacer spacer_prefix="right" parent="base_chassis_link">
+                <origin xyz="0 -0.19582 0" rpy="0 0 ${M_PI}" />
+            </xacro:inv_double_spacer>
+        </xacro:if>
+        <xacro:if value="$(optenv SEGWAY_440_LE_ECI false)">
+            <xacro:eci_440_spacer parent="base_chassis_link">
+                <origin xyz="0 0 0" rpy="0 0 0" />
+            </xacro:eci_440_spacer>
+        </xacro:if>
         <!-- UI Box -->
         <xacro:large_enclosure parent="base_chassis_link">

Commit message: updating to add the 440LE navigator elite package
also fixed the waypoint initialization of the marker array in the segway_ros package

File: segway_description/urdf/RMP_440LE/rmp.urdf.xacro (robot description, xacro)
@@ -32,4 +32,5 @@
     <xacro:include filename="$(find segway_description)/urdf/segway_components/eci_440_spacer.urdf.xacro" />
     <xacro:include filename="$(find segway_description)/urdf/segway_components/large_enclosure.urdf.xacro" />
+    <xacro:include filename="$(find segway_description)/urdf/segway_components/rmp440_le_nave_brackets.urdf.xacro" />
     <xacro:include filename="$(find segway_description)/urdf/accessories.urdf.xacro" />
     <property name="M_PI" value="3.14159"/>
@@ -188,4 +189,9 @@
             </xacro:eci_440_spacer>
         </xacro:if>
+        <xacro:if value="$(optenv HAS_SEGWAY_440_NAVE_PACKAGE false)">
+            <xacro:rmp440_le_nave_brackets parent="base_chassis_link">
+                <origin xyz="0 0 0" rpy="0 0 0" />
+            </xacro:rmp440_le_nave_brackets>
+        </xacro:if>
         <!-- UI Box -->
         <xacro:large_enclosure parent="base_chassis_link">

File: segway_description/urdf/accessories.urdf.xacro (robot description, xacro)
@@ -27,4 +27,5 @@
     <xacro:include filename="$(find segway_description)/urdf/sensors/velodyne_vlp16.urdf.xacro"/>
     <xacro:include filename="$(find segway_description)/urdf/sensors/pgr_flea3.urdf.xacro"/>
+    <xacro:include filename="$(find segway_description)/urdf/sensors/garmin_18x_lvc_gps.urdf.xacro"/>
     <property name="M_PI" value="3.14159"/>
     <xacro:macro name="segway_accessories">
@@ -54,24 +55,7 @@
         <!--GPS Link-->
         <xacro:if value="$(optenv SEGWAY_HAS_GPS false)">
-            <link name="gps_frame"/>
-            <joint name="gps_joint" type="fixed">
-                <origin xyz="$(optenv GPS_XYZ -0.1189 0 0.34665)" rpy="$(optenv GPS_RPY 0 0 0)" />
-                <parent link="$(optenv SEGWAY_PARENT_LINK base_chassis_link)" />
-                <child link="gps_frame" />
-            </joint>
-            <gazebo>
-                <plugin name="gps_controller" filename="libhector_gazebo_ros_gps.so">
-                    <alwaysOn>1</alwaysOn>
-                    <updateRate>40</updateRate>
-                    <bodyName>gps_frame</bodyName>
-                    <topicName>/segway/feedback/gps/fix_2d</topicName>
-                    <velocityTopicName>/segway/feedback/gps/vel</velocityTopicName>
-                    <referenceLatitude>40.712784</referenceLatitude>
-                    <referenceLongitude>-74.005941</referenceLongitude>
-                    <referenceHeading>0</referenceHeading>
-                    <referenceAltitude>0</referenceAltitude>
-                    <drift>0.0001 0.0001 0.0001</drift>
-                </plugin>
-            </gazebo>
+            <xacro:garmin_18x_lvc_gps parent="$(optenv SEGWAY_PARENT_LINK base_chassis_link)">
+                <origin xyz="$(optenv GPS_XYZ 0 0 1.0)" rpy="$(optenv GPS_RPY 0 0 3.1416)" />
+            </xacro:garmin_18x_lvc_gps>
         </xacro:if>
         <!-- RGBD Sensor -->
