Commit message: update for kinetic

File: segway_description/urdf/NAVIGATOR_ELITE/rmp.urdf.xacro (robot description, xacro)
@@ -30,5 +30,5 @@
     <xacro:include filename="$(find segway_description)/urdf/segway_components/navigator_ui.urdf.xacro" />
     <xacro:include filename="$(find segway_description)/urdf/accessories.urdf.xacro" />
-    <property name="M_PI" value="3.14159"/>
+    <xacro:property name="M_PI" value="3.14159"/>
     <!-- Wheel Mounting Positions -->
     <xacro:property name="track" value="0.542391" />

File: segway_description/urdf/RMP_110/rmp.urdf.xacro (robot description, xacro)
@@ -30,5 +30,5 @@
     <xacro:include filename="$(find segway_description)/urdf/segway_components/hmi_plate_110.urdf.xacro" />
     <xacro:include filename="$(find segway_description)/urdf/accessories.urdf.xacro" />
-    <property name="M_PI" value="3.14159"/>
+    <xacro:property name="M_PI" value="3.14159"/>
     <!-- Wheel Mounting Positions -->
     <xacro:property name="track" value="0.48122440" />

File: segway_description/urdf/RMP_110_WIDE/rmp.urdf.xacro (robot description, xacro)
@@ -30,5 +30,5 @@
     <xacro:include filename="$(find segway_description)/urdf/segway_components/navigator_ui_box_110.urdf.xacro" />
     <xacro:include filename="$(find segway_description)/urdf/accessories.urdf.xacro" />
-    <property name="M_PI" value="3.14159"/>
+    <xacro:property name="M_PI" value="3.14159"/>
     <!-- Wheel Mounting Positions -->
     <xacro:property name="track" value="0.542391" />

File: segway_description/urdf/RMP_210/rmp.urdf.xacro (robot description, xacro)
@@ -31,5 +31,5 @@
     <xacro:include filename="$(find segway_description)/urdf/segway_components/ui_box_spacer_mount.urdf.xacro" />
     <xacro:include filename="$(find segway_description)/urdf/accessories.urdf.xacro" />
-    <property name="M_PI" value="3.14159"/>
+    <xacro:property name="M_PI" value="3.14159"/>
     <!-- Wheel Mounting Positions -->
     <xacro:property name="track" value="0.542391" />

File: segway_description/urdf/RMP_220/rmp.urdf.xacro (robot description, xacro)
@@ -31,5 +31,5 @@
     <xacro:include filename="$(find segway_description)/urdf/segway_components/ui_box.urdf.xacro" />
     <xacro:include filename="$(find segway_description)/urdf/accessories.urdf.xacro" />
-    <property name="M_PI" value="3.14159"/>
+    <xacro:property name="M_PI" value="3.14159"/>
     <!-- Wheel Mounting Positions -->
     <xacro:property name="track" value="0.542391" />

File: segway_description/urdf/RMP_440LE/rmp.urdf.xacro (robot description, xacro)
@@ -34,5 +34,5 @@
     <xacro:include filename="$(find segway_description)/urdf/segway_components/rmp440_le_nave_brackets.urdf.xacro" />
     <xacro:include filename="$(find segway_description)/urdf/accessories.urdf.xacro" />
-    <property name="M_PI" value="3.14159"/>
+    <xacro:property name="M_PI" value="3.14159"/>
     <!-- Wheel Mounting Positions -->
     <xacro:property name="wheel_track" value="$(optenv SEGWAY_440LE_WHEEL_TRACK 0.66067)" />

File: segway_description/urdf/RMP_440SE/rmp.urdf.xacro (robot description, xacro)
@@ -30,5 +30,5 @@
     <xacro:include filename="$(find segway_description)/urdf/segway_components/ui_box_spacer_mount.urdf.xacro" />
     <xacro:include filename="$(find segway_description)/urdf/accessories.urdf.xacro" />
-    <property name="M_PI" value="3.14159"/>
+    <xacro:property name="M_PI" value="3.14159"/>
     <!-- Wheel Mounting Positions -->
     <xacro:property name="wheel_track" value="0.66067" />

File: segway_description/urdf/RMP_OMNI/rmp.urdf.xacro (robot description, xacro)
@@ -33,5 +33,5 @@
     <xacro:include filename="$(find segway_description)/urdf/segway_components/ui_box.urdf.xacro" />
     <xacro:include filename="$(find segway_description)/urdf/accessories.urdf.xacro" />
-    <property name="M_PI" value="3.14159"/>
+    <xacro:property name="M_PI" value="3.14159"/>
     <!-- Wheel Mounting Positions -->
     <xacro:property name="wheel_track" value="0.693251" />
