Commit message: updating for new configuration layout to allow sim

File: segway_description/urdf/accessories.urdf.xacro (robot description, xacro)
@@ -42,5 +42,5 @@
                     <updateRate>50.0</updateRate>
                     <bodyName>ext_imu_frame</bodyName>
-                    <topicName>/segway/feedback/um7_imu</topicName>
+                    <topicName>/segway/feedback/ext_imu</topicName>
                     <accelDrift>0.005 0.005 0.005</accelDrift>
                     <accelGaussianNoise>0.005 0.005 0.005</accelGaussianNoise>
@@ -54,9 +54,9 @@
         <!--GPS Link-->
         <xacro:if value="$(optenv SEGWAY_HAS_GPS false)">
-            <link name="gps_link"/>
+            <link name="gps_frame"/>
             <joint name="gps_joint" type="fixed">
                 <origin xyz="$(optenv GPS_XYZ -0.1189 0 0.34665)" rpy="$(optenv GPS_RPY 0 0 0)" />
                 <parent link="$(optenv SEGWAY_PARENT_LINK base_chassis_link)" />
-                <child link="gps_link" />
+                <child link="gps_frame" />
             </joint>
             <gazebo>
@@ -64,6 +64,6 @@
                     <alwaysOn>1</alwaysOn>
                     <updateRate>40</updateRate>
-                    <bodyName>gps_link</bodyName>
-                    <topicName>/segway/feedback/gps/fix</topicName>
+                    <bodyName>gps_frame</bodyName>
+                    <topicName>/segway/feedback/gps/fix_2d</topicName>
                     <velocityTopicName>/segway/feedback/gps/vel</velocityTopicName>
                     <referenceLatitude>40.712784</referenceLatitude>

Commit message: updates from sim testing

File: segway_description/urdf/accessories.urdf.xacro (robot description, xacro)
@@ -103,7 +103,7 @@
             <xacro:pgr_flea3 camera_prefix="camera" parent="$(optenv SEGWAY_PARENT_LINK base_chassis_link)"
                           image_format="R8G8B8" image_topic_name="image_raw"
-                          camera_info_topic_name="camera_info" hfov="90" focal_length="320.000105"
+                          camera_info_topic_name="camera_info" hfov="90" focal_length="317.772992"
                           hack_baseline="0" image_width="640" image_height="480">
-                <origin xyz="$(optenv FLEA3_XYZ 0 0 0.32739)" rpy="$(optenv FLEA3_RPY -1.5708 0 -1.5708)" />
+                <origin xyz="$(optenv FLEA3_XYZ 0 0 0.32739)" rpy="$(optenv FLEA3_RPY 0 0 0)" />
             </xacro:pgr_flea3>
         </xacro:if>

File: segway_description/urdf/sensors/velodyne_vlp16.urdf.xacro (robot description, xacro)
@@ -81,5 +81,5 @@
                 <plugin name="plugin_1" filename="libgazebo_ros_block_laser.so">
                     <updateRate>10.0</updateRate>
-                    <topicName>/segway/velodyne_scan</topicName>
+                    <topicName>/velodyne_pointcloud</topicName>
                     <frameName>/segway/velodyne_frame</frameName>
                 </plugin>

Commit message: updating the SICK laser to use TIM which is now standard; fixed BSA data not propegating; fixed file permissions that accidentally changed to +x;

File: segway_description/urdf/accessories.urdf.xacro (robot description, xacro)
@@ -23,5 +23,5 @@
 <robot name="segway_accessories" xmlns:xacro="http://ros.org/wiki/xacro">
     <xacro:include filename="$(find segway_description)/urdf/sensors/rgbd_sensor.urdf.xacro"/>
-    <xacro:include filename="$(find segway_description)/urdf/sensors/sick_lms1xx.urdf.xacro"/>
+    <xacro:include filename="$(find segway_description)/urdf/sensors/sick_tim.urdf.xacro"/>
     <xacro:include filename="$(find segway_description)/urdf/sensors/hokuyo_ust20lx.urdf.xacro"/>
     <xacro:include filename="$(find segway_description)/urdf/sensors/velodyne_vlp16.urdf.xacro"/>
@@ -81,9 +81,9 @@
             </xacro:rgbd_sensor>
         </xacro:if>
-        <!-- SICK LMS1XX Sensor -->
-        <xacro:if value="$(optenv SEGWAY_HAS_SICK false)">
-            <xacro:sick_lms1xx laser_prefix="base" parent="$(optenv SEGWAY_PARENT_LINK base_chassis_link)">
-                <origin xyz="$(optenv SICK_LMS1XX_XYZ 0 0 1.0)" rpy="$(optenv SICK_LMS1XX_RPY 3.1416 0 0)" />
-            </xacro:sick_lms1xx>
+        <!-- SICK TIM Sensor -->
+        <xacro:if value="$(optenv SEGWAY_HAS_SICK_TIM false)">
+            <xacro:sick_tim laser_prefix="base" parent="$(optenv SEGWAY_PARENT_LINK base_chassis_link)">
+                <origin xyz="$(optenv SICK_TIM_XYZ 0 0 1.0)" rpy="$(optenv SICK_TIM_RPY 3.1416 0 0)" />
+            </xacro:sick_tim>
         </xacro:if>
         <!-- Hokuyo UST-20LX Sensor -->

Commit message: adding support for 2 lasers

File: segway_description/urdf/accessories.urdf.xacro (robot description, xacro)
@@ -81,15 +81,31 @@
             </xacro:rgbd_sensor>
         </xacro:if>
-        <!-- SICK TIM Sensor -->
-        <xacro:if value="$(optenv SEGWAY_HAS_SICK_TIM false)">
-            <xacro:sick_tim laser_prefix="base" parent="$(optenv SEGWAY_PARENT_LINK base_chassis_link)">
-                <origin xyz="$(optenv SICK_TIM_XYZ 0 0 1.0)" rpy="$(optenv SICK_TIM_RPY 3.1416 0 0)" />
-            </xacro:sick_tim>
+        <!-- First laser Sensor -->
+        <xacro:if value="$(optenv SEGWAY_HAS_ONE_2D_LASER false)">
+            <!-- SICK TIM Sensor -->
+            <xacro:if value="$(optenv SEGWAY_LASER1_IS_SICK_TIM false)">
+                <xacro:sick_tim laser_prefix="$(optenv LASER1_PREFIX base)" parent="$(optenv SEGWAY_PARENT_LINK base_chassis_link)">
+                    <origin xyz="$(optenv LASER1_XYZ 0.35 0 0.2)" rpy="$(optenv LASER1_RPY 3.14159 0 0)" />
+                </xacro:sick_tim>
+            </xacro:if>
+            <xacro:if value="$(optenv SEGWAY_LASER1_IS_HOKUYO false)">
+                <xacro:hokuyo_ust20lx laser_prefix="$(optenv LASER1_PREFIX base)" parent="$(optenv VECTOR_PARENT_LINK base_chassis_link)">
+                    <origin xyz="$(optenv LASER1_XYZ 0.35 0 0.2)" rpy="$(optenv LASER1_RPY 3.14159 0 0)" />
+                </xacro:hokuyo_ust20lx>
+            </xacro:if>
         </xacro:if>
-        <!-- Hokuyo UST-20LX Sensor -->
-        <xacro:if value="$(optenv SEGWAY_HAS_HOKUYO false)">
-            <xacro:hokuyo_ust20lx laser_prefix="base" parent="$(optenv SEGWAY_PARENT_LINK base_chassis_link)">
-                <origin xyz="$(optenv HOKUYO_XYZ 0.35 0 0.1)" rpy="$(optenv HOKUYO_RPY 0 0 0)" />
-            </xacro:hokuyo_ust20lx>
+        <!-- Second laser Sensor -->
+        <xacro:if value="$(optenv SEGWAY_HAS_SECOND_2D_LASER false)">
+            <!-- SICK TIM Sensor -->
+            <xacro:if value="$(optenv SEGWAY_LASER2_IS_SICK_TIM false)">
+                <xacro:sick_tim laser_prefix="$(optenv LASER2_PREFIX base)" parent="$(optenv SEGWAY_PARENT_LINK base_chassis_link)">
+                    <origin xyz="$(optenv LASER2_XYZ 0.35 0 0.2)" rpy="$(optenv LASER2_RPY 3.14159 0 0)" />
+                </xacro:sick_tim>
+            </xacro:if>
+            <xacro:if value="$(optenv SEGWAY_LASER2_IS_HOKUYO false)">
+                <xacro:hokuyo_ust20lx laser_prefix="$(optenv LASER2_PREFIX base)" parent="$(optenv VECTOR_PARENT_LINK base_chassis_link)">
+                    <origin xyz="$(optenv LASER2_XYZ 0.35 0 0.2)" rpy="$(optenv LASER2_RPY 3.14159 0 0)" />
+                </xacro:hokuyo_ust20lx>
+            </xacro:if>
         </xacro:if>
         <!-- Velodyne VLP-16 Sensor -->

Commit message: melodic

File: segway_description/urdf/accessories.urdf.xacro (robot description, xacro)
@@ -96,5 +96,5 @@
         <xacro:if value="$(optenv SEGWAY_HAS_VLP16 false)">
             <xacro:velodyne_vlp16 parent="$(optenv SEGWAY_PARENT_LINK base_chassis_link)">
-                <origin xyz="$(optenv VLP16_XYZ 0 0 0.39991)" rpy="$(optenv VLP16_RPY 0 0 0)" />
+                <origin xyz="$(optenv VLP16_XYZ 0 0 0.42760744)" rpy="$(optenv VLP16_RPY 0 0 0)" />
             </xacro:velodyne_vlp16>
         </xacro:if>
